Commit message: updated to work with diff drive

File: src/my_robot/urdf/my_robot.xacro (robot description, xacro)
@@ -22,17 +22,15 @@
     <xacro:property name="Rod_z" value="${wheel_radius/2}" />
     <!-- Front left and right wheel rods -->
-    <joint name="left_steer_joint" type="revolute">
+    <joint name="left_steer_joint" type="fixed">
         <parent link="base_link" />
         <child link="front_left_rod_steer" />
         <origin xyz="${Rod_x} ${Rod_y} ${Rod_z}" rpy="0.0 0.0 0.0" />
         <axis xyz="0.0 0.0 1.0" />
-        <limit effort="100.0" lower="-1.0" upper="1.0" velocity="10.0" />
     </joint>
-    <joint name="right_steer_joint" type="revolute">
+    <joint name="right_steer_joint" type="fixed">
         <parent link="base_link" />
         <child link="front_right_rod_steer" />
         <origin xyz="${Rod_x} ${-Rod_y} ${Rod_z}" rpy="0.0 0.0 0.0" />
         <axis xyz="0.0 0.0 1.0" />
-        <limit effort="100.0" lower="-1.0" upper="1.0" velocity="10.0" />
     </joint>
     <!-- Front left and right wheels -->
@@ -75,12 +73,3 @@
         <axis xyz="0.0 1.0 0.0" />
     </joint>
-    <!-- lidar joint -->
-    <!--
-    <joint name="lidar_joint" type="fixed">
-        <parent link="base_link" />
-        <child link="lidar_link" />
-        <origin xyz="${lidar_x} 0 ${lidar_z}" rpy="0.0 0.0 0.0" />
-        <axis xyz="0 0 0" />
-    </joint> -->
-    <!-- <xacro:robot_gazebo_plugin /> -->
 </robot>

File: src/my_robot/urdf/plugins.xacro (robot description, xacro)
@@ -3,13 +3,10 @@
     <gazebo>
         <plugin
-            filename="gz-sim-ackermann-steering-system"
-            name="gz::sim::systems::AckermannSteering">
+            filename="gz-sim-diff-drive-system"
+            name="gz::sim::systems::DiffDrive">
             <left_joint>back_left_wheel_joint</left_joint>
             <right_joint>back_right_wheel_joint</right_joint>
             <left_joint>front_left_wheel_joint</left_joint>
             <right_joint>front_right_wheel_joint</right_joint>
-            <left_steering_joint>left_steer_joint</left_steering_joint>
-            <right_steering_joint>right_steer_joint</right_steering_joint>
-            <steer_p_gain>10</steer_p_gain>
             <topic>cmd_vel</topic>
             <odom_topic>odom</odom_topic>
